File: pcb/argb_controller.kicad_pcb (KiCad board)
At the start: 2 copper layers, 51.5 x 106.5 mm, 14 parts, among them U1 74AHCT125, U3 XIAO-RP2040-DIP

Commit message: Add files via upload
Routing:
- net GND: track 349.3 -> 368.1 mm
- net D2: track 63.5 -> 64.9 mm
- added copper zone on B.Cu, net GND
